Commit message: edit urdfddd

File: description/robot_core.xacro (robot description, xacro)
@@ -128,5 +128,5 @@
         </collision>
         <xacro:inertial_sphere mass="0.1" radius="0.033">
-            <origin xyz="0 0 0" rpy="0 0 0"/>
+            <origin xyz="0 1 0" rpy="0 0 0"/>
         </xacro:inertial_sphere>
     </link>

Commit message: Edit core URDF

File: description/robot_core.xacro (robot description, xacro)
@@ -128,5 +128,5 @@
         </collision>
         <xacro:inertial_sphere mass="0.1" radius="0.033">
-            <origin xyz="0 1 0" rpy="0 0 0"/>
+            <origin xyz="0 0 0" rpy="0 0 0"/>
         </xacro:inertial_sphere>
     </link>

Commit message: Created Gazebo Plugins and World

File: description/robot_core.xacro (robot description, xacro)
@@ -41,4 +41,7 @@
         </xacro:inertial_box>
     </link>
+    <gazebo reference="chassis">
+        <material>Gazebo/White</material>
+    </gazebo>
     <!-- LEFT WHEEL LINK -->
     <joint name="left_wheel_joint" type="continuous">
@@ -64,4 +67,7 @@
         </xacro:inertial_cylinder>
     </link>
+    <gazebo reference="left_wheel">
+        <material>Gazebo/Blue</material>
+    </gazebo>
     <!-- RIGHT WHEEL LINK -->
     <joint name="right_wheel_joint" type="continuous">
@@ -87,4 +93,7 @@
         </xacro:inertial_cylinder>
     </link>
+    <gazebo reference="right_wheel">
+        <material>Gazebo/Blue</material>
+    </gazebo>
     <!-- LEFT CASTER WHEEL LINK -->
     <joint name="left_caster_wheel_joint" type="fixed">
@@ -109,4 +118,9 @@
         </xacro:inertial_sphere>
     </link>
+    <gazebo reference="left_caster_wheel">
+        <material>Gazebo/Black</material>
+        <mu1 value="0.001"/>
+        <mu2 value="0.001"/>
+    </gazebo>
     <!-- RIGHT CASTER WHEEL LINK -->
     <joint name="right_caster_wheel_joint" type="fixed">
@@ -131,3 +145,8 @@
         </xacro:inertial_sphere>
     </link>
+    <gazebo reference="right_caster_wheel">
+        <material>Gazebo/Black</material>
+        <mu1 value="0.001"/>
+        <mu2 value="0.001"/>
+    </gazebo>
 </robot>

Commit message: Update robot_core.xacro

File: description/robot_core.xacro (robot description, xacro)
@@ -25,5 +25,5 @@
     <link name="chassis">
         <visual>
-            <origin xyz="0.205 0 0.1"/> <!--half of box size-->
+            <origin xyz="0.205 0 0.1"/> <!--half value of box size -->
             <geometry>
                 <box size="0.41 0.37 0.20"/>
